Commit message: Update simulation for road shoulder weeding with convoy formation
Scenario change: farm field → road shoulder (路肩) weeding
Robot formation: side-by-side → convoy column along road (縦列隊形)

Changes:
- road_shoulder.sdf: New 40m road world with asphalt (Y=-4~+4), shoulder
  surface (Y=+4~+7.5), curb, 10 guardrail posts+beam, road markings
  (centerline/edge lines), angled overhead camera view
- farm_sim.launch.py: Switch world to road_shoulder.sdf; robots now spawn
  in column at Y=5.5 (shoulder center) facing +X (road direction):
  Robot1 x=-4, Robot2 x=-8, Robot3 x=-12 (4m spacing)
- robot2_weeder.urdf.xacro: Move RGBD camera and weeder blade to left side
  (+Y direction) to face the outer shoulder where weeds grow
- spawn_weeds.py: Restrict weed spawning to shoulder area only
  (X=-18~+18m, Y=4.5~7.0m); exclude circles around robot start positions
- display.rviz: New RViz2 config with Grid/RobotModel/TF displays and
  Fixed Frame set to robot1/base_link for correct URDF visualization
- display.launch.py: Simplified; loads display.rviz automatically so
  robot model appears on launch without manual RViz configuration
- CMakeLists.txt (farm_description): Re-add config/ to install targets

https://claude.ai/code/session_01FyqdRzg54CjceHKaqJRyWt

File: farm_swarm_ws/src/farm_description/urdf/robot2_weeder.urdf.xacro (robot description, xacro)
@@ -2,7 +2,11 @@
 <!--
   Robot ② 除草ロボット (Weeder)
+  路肩除草想定:
+    - ロボットはX軸+方向に進行 (道路方向)
+    - 路肩は進行方向左側 (+Y方向) に展開
+    - RGBDカメラと除草刃は左側面 (+Y方向) に搭載
   搭載センサ・機器:
-    - RealSense D435 RGBD (右側面: 雑草検出)
-    - 回転除草刃 (右側面下部)
+    - RealSense D435 RGBD (左側面: 雑草検出)
+    - 回転除草刃 (左側面下部)
   役割: 雑草検出・除草機駆動
 -->
@@ -12,16 +16,16 @@
   <!-- 差動駆動台車 (緑色) -->
   <xacro:diff_drive_base robot_name="robot2" color="green"/>
-  <!-- 右側方RGBD: 除草対象検出用 -->
+  <!-- 左側方RGBD: 路肩方向 (+Y) の除草対象検出用 -->
   <xacro:realsense_d435
     prefix="robot2_side"
     parent="robot2/base_link"
-    xyz="0.0 -0.20 0.12"
-    rpy="0.0 0.3 ${-PI/2}"
+    xyz="0.0 0.20 0.12"
+    rpy="0.0 0.3 ${PI/2}"
     robot="robot2"/>
-  <!-- 除草機構: 回転刃 (右側面下部) -->
+  <!-- 除草機構: 回転刃 (左側面下部, 路肩方向) -->
   <joint name="robot2/weeder_joint" type="continuous">
     <parent link="robot2/base_link"/>
     <child  link="robot2/weeder_blade"/>
-    <origin xyz="0.05 -0.28 -0.04" rpy="0.0 0.0 0.0"/>
+    <origin xyz="0.05 0.28 -0.04" rpy="0.0 0.0 0.0"/>
     <axis xyz="0 0 1"/>
     <dynamics damping="0.05"/>
@@ -47,5 +51,4 @@
     </inertial>
   </link>
-  <!-- 除草刃ジョイント状態を追加でパブリッシュ -->
   <gazebo>
     <plugin filename="gz-sim-joint-state-publisher-system"

Commit message: Add autonomous navigation: Robot① obstacle avoidance, Robot②③ convoy following
- robot1_navigator_node: reactive obstacle avoidance (LaserScan front sector),
  lane keeping at Y=5.5 (P-control), auto U-turn at X=±17m, cruise 0.6m/s
- convoy_controller_node: go-to-goal control for Robot②③ following 4m behind
  leader, max 0.7m/s, heading-weighted linear velocity scaling
- boundary_enforcer: simplified to danger zone only (no warn zone),
  avoids conflict with autonomous navigation nodes
- robot2 URDF: move blade and camera to -Y side (toward road/shoulder boundary)
- weed_removal_node: update blade offset Y to -0.28m (road-boundary side)
- spawn_weeds: update Y range to [4.1, 5.4] (inner shoulder near road edge)
- perception.launch: add robot1_navigator and convoy_controller nodes

https://claude.ai/code/session_01FyqdRzg54CjceHKaqJRyWt

File: farm_swarm_ws/src/farm_description/urdf/robot2_weeder.urdf.xacro (robot description, xacro)
@@ -4,9 +4,10 @@
   路肩除草想定:
     - ロボットはX軸+方向に進行 (道路方向)
-    - 路肩は進行方向左側 (+Y方向) に展開
-    - RGBDカメラと除草刃は左側面 (+Y方向) に搭載
+    - ロボットは路肩 (Y=5.5) を走行
+    - 雑草は路肩内側 (道路との境目、Y≈4〜5.5) に生育
+    - RGBDカメラと除草刃は右側面 (-Y方向、道路境界側) に搭載
   搭載センサ・機器:
-    - RealSense D435 RGBD (左側面: 雑草検出)
-    - 回転除草刃 (左側面下部)
+    - RealSense D435 RGBD (右側面: 雑草検出)
+    - 回転除草刃 (右側面下部)
   役割: 雑草検出・除草機駆動
 -->
@@ -16,16 +17,16 @@
   <!-- 差動駆動台車 (緑色) -->
   <xacro:diff_drive_base robot_name="robot2" color="green"/>
-  <!-- 左側方RGBD: 路肩方向 (+Y) の除草対象検出用 -->
+  <!-- 右側方RGBD: 道路境界方向 (-Y) の除草対象検出用 -->
   <xacro:realsense_d435
     prefix="robot2_side"
     parent="robot2/base_link"
-    xyz="0.0 0.20 0.12"
-    rpy="0.0 0.3 ${PI/2}"
+    xyz="0.0 -0.20 0.12"
+    rpy="0.0 0.3 ${-PI/2}"
     robot="robot2"/>
-  <!-- 除草機構: 回転刃 (左側面下部, 路肩方向) -->
+  <!-- 除草機構: 回転刃 (右側面下部, 道路境界方向) -->
   <joint name="robot2/weeder_joint" type="continuous">
     <parent link="robot2/base_link"/>
     <child  link="robot2/weeder_blade"/>
-    <origin xyz="0.05 0.28 -0.04" rpy="0.0 0.0 0.0"/>
+    <origin xyz="0.05 -0.28 -0.04" rpy="0.0 0.0 0.0"/>
     <axis xyz="0 0 1"/>
     <dynamics damping="0.05"/>
